File: electronics/rover/pmu.sch (EAGLE design)
At the start: 41 parts, among them U1 L5973D, U2 L5973D, U3 L5973D

Commit message: Added new electronic designs
Parts:
- removed C10: 22n, SparkFun-Passives:CAP0805
- removed C11: 330u, rcl:CPOL-USE
- removed C12: 220p, SparkFun-Passives:CAP0805
- removed C9: 10u, SparkFun-Passives:CAP1210
- removed D5: (no value), SparkFun-DiscreteSemi:DIODESMB
- removed D6: GREEN, SparkFun-LED:LED-GREENLARGE
- removed L3: 15uH, Panasonic-ELL:ELL8TP150MB-8TP
- removed MCU_PWR: (no value), SparkFun-Connectors:M05PTH
- removed R10: 8.2k, SparkFun-Passives:RESISTOR0805-RES
- removed R11: 2.7k, SparkFun-Passives:RESISTOR0805-RES
- removed R12: 330, SparkFun-Passives:RESISTOR0805-RES
- removed R9: 4k7, SparkFun-Passives:RESISTOR0805-RES
- removed U3: L5973D, L5973D:L5973D
- added JP1: (no value), SparkFun-Connectors:M04PTH
- C3, C7: device rcl:CPOL-USE -> SparkFun-Passives:CAP_POL7343
- D2, D4: device SparkFun-LED:LED-GREENLARGE -> led:LEDCHIP-LED0805
Connections:
- removed net 5VS: C11.+, L3.1, MCU_PWR.2, R10.2, R12.2
- removed net N$13: C10.2, R9.1
- removed net N$14: D5.C, L3.2, U3.OUT
- removed net N$15: R10.1, R11.2, U3.FB
- removed net N$16: D6.A, R12.1
- removed net N$19: U3.VREF
- removed net N$7: C10.1, C12.1, U3.COMP
- net 3.3V: now also JP1.2; no longer MCU_PWR.3
- net 5V: now also JP1.3; no longer MCU_PWR.4
- net GND: now also JP1.1; no longer C11.-, C12.2, C9.2, D5.A, D6.C, MCU_PWR.1, R11.1, R9.2, U3.EXPOSED_PAD, U3.GND, U3.INH
- net V_BATT: now also JP1.4; no longer C9.1, MCU_PWR.5, U3.VCC
Other:
- note added: "+3.3V Regulator"
- note added: "+5V Regulator"
- note added: "Battery"
- note added: "To CPU"
- note added: "To MCU"
- moved on the sheet: BATT, C1, C2, C3, C4, C5, C6, C7, C8, CPU_PWR, D1, D2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
