File: electronics/rover/old (rev a)/mcu.sch (EAGLE design)
At the start: 34 parts, among them IC1 24LC128SM, IC2 24LC128SM, J1 AVR_SPI_PRG_62X3_LOCK, M1 M02PTH, M2 M02PTH, Q2 16M, U1 DRV8833_PWP_16, U2 MPL3115A2LGA8, U4 ATMEGA328P

Commit message: Added new electronic designs
Parts:
- removed C3, C4: 100nF, SparkFun-Capacitors:1UF-25V-10%(0805)
- removed C5: 1u, SparkFun-Passives:CAP0805
- removed POD: (no value), SparkFun-Connectors:M03PTH
- removed R2: 4.7k, SparkFun-Passives:RESISTOR0805-RES
- removed R3: 22k, SparkFun-Passives:RESISTOR0805-RES
- removed R4: 10k, SparkFun-Passives:RESISTOR0805-RES
- removed U2: MPL3115A2LGA8, SparkFun-Sensors:MPL3115A2LGA8
- added JP3: (no value), SparkFun-Connectors:M03LOCK_LONGPADS
- added MCU_PWR: (no value), SparkFun-Connectors:M05PTH
- added MSW: (no value), SparkFun-Connectors:M03LONGPADS
- added R16, R17: 10k, SparkFun-Passives:RESISTOR0805-RES
- added R18, R19: 100, SparkFun-Passives:RESISTOR0805-RES
- added TPS: (no value), SparkFun-Connectors:M06LOCK
- CPU: device SparkFun-Connectors:M05PTH -> SparkFun-Connectors:M05PTH_LONGPADS
- JP1, M1, M2: value M02PTH -> M02PTH3; device SparkFun-Connectors:M02PTH -> SparkFun-Connectors:M02PTH3
- JP2: device SparkFun-Connectors:M04PTH -> SparkFun-Connectors:M03LOCK_LONGPADS
Connections:
- net AIS renamed N$25
- net BIS renamed N$24
- net ISP_MISO renamed N$19
- net ISP_SCK renamed N$18
- net STAT_LED renamed N$1
- net VCP renamed N$21
- net VINT renamed N$23
- removed net CAP: C4.2, U2.CAP
- removed net ISP_MOSI: J1.4, U4.PB3(MOSI/OC2)
- removed net LNK_RST: C3.1, CPU.3
- removed net MON: R3.1, R4.2, U4.PC0(ADC0)
- removed net POD_MISO: POD.2, U4.PD4(XCK/T0)
- removed net POD_MOSI: POD.1, U4.PB0(ICP)
- new net 5VS: JP2.2, JP3.2, MCU_PWR.2
- new net FLT: U1.NFAULT, U4.PC3(ADC3)
- new net N$17: JP2.1, R18.2
- new net N$20: JP3.1, R19.2
- new net SERVO1: R18.1, U4.PD4(XCK/T0)
- new net SERVO2: R19.1, U4.PD5(T1)
- new net SW1: MSW.1, R16.1, U4.PD2(INT0)
- new net SW2: MSW.3, R17.1, U4.PD3(INT1)
- net 3.3V: now also MCU_PWR.3, TPS.1; no longer C5.1, JP2.2, U2.VDD, U2.VDDIO
- net 5V: now also MCU_PWR.4, R16.2, R17.2; no longer JP2.3
- net GND: now also JP2.3, JP3.3, MCU_PWR.1, MSW.2, TPS.6; no longer C4.1, C5.2, JP2.1, POD.3, R2.1, R4.1, U2.GND
- net M2B_CTL: now also J1.4, U4.PB3(MOSI/OC2); no longer U4.PD5(T1)
- net RDY: no longer R2.2
- net RST: now also CPU.3; no longer C3.2
- net SCL: now also TPS.3; no longer U2.SCL
- net SDA: now also TPS.2; no longer U2.SDA
- net V_BATT: now also MCU_PWR.5; no longer JP2.4, R3.2
Other:
- note removed: "ATmega"
- note removed: "EEPROMs"
- note removed: "ISP"
- note removed: "LED"
- note removed: "Landing Module Link"
- note removed: "Motor Driver"
- note removed: "Piezo"
- note removed: "Power Input"
- note removed: "Pressure Sensor"
- note removed: "To CPU Board"
- moved on the sheet: C1, C13, C14, C15, C16, C17, C18, C2, CPU, IC1, IC2, JP1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
